Commit message: js added

File: config/ruka.urdf (robot description, URDF)
Before this commit: robot ruka, 12 links, 11 joints
Joints:
- joint link_02__link_03: origin xyz=0 0.28 0 rpy=0 0 1.57 -> xyz=0 0.28 0 rpy=0 0 3.14

Commit message: soft limits added

File: config/ruka.urdf (robot description, URDF)
Before this commit: robot ruka, 12 links, 11 joints
Joints:
- joint base_link__link_01: limit lower=-3.14 upper=3.14 effort=1000.0 velocity=0.5 -> lower=-2.96 upper=2.96 effort=1000.0 velocity=0.5
- joint link_01__link_02: limit lower=-3.14 upper=3.14 effort=1000.0 velocity=0.5 -> lower=-3.57 upper=0 effort=1000.0 velocity=0.5; origin xyz=0.01 0 0.179 rpy=1.57 0 0 -> xyz=0.01 0 0.179 rpy=1.57 -1.57 0
- joint link_02__link_03: limit lower=-3.14 upper=3.14 effort=1000.0 velocity=0.5 -> lower=0.035 upper=5.23 effort=1000.0 velocity=0.5; origin xyz=0 0.28 0 rpy=0 0 3.14 -> xyz=0 0.28 0 rpy=0 0 0.0175
- joint link_03__link_04: limit lower=-3.14 upper=3.14 effort=1000.0 velocity=0.5 -> lower=-2.87 upper=2.87 effort=1000.0 velocity=0.5
- joint link_04__link_05: limit lower=-3.14 upper=3.14 effort=1000.0 velocity=0.5 -> lower=-2.44 upper=2.44 effort=1000.0 velocity=0.5
