Commit message: update

File: config/imu.ros2_control.xacro (robot description, xacro)
@@ -3,9 +3,4 @@
   <xacro:macro name="ruka_ros2_sensor" params="name prefix use_mock_hardware:=^|true mock_sensor_commands:=^|false">
     <ros2_control name="${name}" type="sensor">
-  <!--   <hardware>
-                 By default, set up controllers for simulation. This won't work on real hardware
-                <plugin>ruka/RukaSensor</plugin>
-      </hardware>
-      -->
       <hardware>
           <plugin>ruka/RukaSensor</plugin>
@@ -15,12 +10,6 @@
        -->
       </hardware>
-<!--
-      <sensor name="x">
-        <state_interface name="orientation.x"/>
-	<param name="frame_id">link_06</param>
-      </sensor>
-       -->
-      <sensor name="${prefix}imu_sensor">
-        <state_interface name="orientation.x"/>
+        <sensor name="${prefix}imu_sensor">
+                <state_interface name="orientation.x"/>
         <state_interface name="orientation.y"/>
         <state_interface name="orientation.z"/>
@@ -32,20 +21,5 @@
         <state_interface name="linear_acceleration.y"/>
         <state_interface name="linear_acceleration.z"/>
-       <!--
-        <state_interface name="force.y"/>
-        <state_interface name="force.z"/>
-        <state_interface name="torque.x"/>
-        <state_interface name="torque.y"/>
-        <state_interface name="torque.z"/>
-        -->
         <param name="frame_id">link_06</param>
-       <!--
-        <param name="fx_range">100</param>
-        <param name="fy_range">100</param>
-        <param name="fz_range">100</param>
-        <param name="tx_range">15</param>
-        <param name="ty_range">15</param>
-        <param name="tz_range">15</param>
-        -->
       </sensor>
     </ros2_control>

File: config/ruka.urdf (robot description, URDF)
Before this commit: robot ruka, 12 links, 11 joints
Joints:
- joint link_01__link_02: limit lower=-3.57 upper=0 effort=1000.0 velocity=0.5 -> lower=-3.57 upper=0.05 effort=1000.0 velocity=0.5
- joint link_02__link_03: limit lower=0.035 upper=5.23 effort=1000.0 velocity=0.5 -> lower=-0.035 upper=5.23 effort=1000.0 velocity=0.5

File: config/ruka.urdf.xacro (robot description, xacro)
@@ -3,5 +3,5 @@
     <xacro:arg name="prefix" default="" />
     <xacro:arg name="initial_positions_file" default="initial_positions.yaml" />
-    <!-- Import ruka urdf file -->
+    <!-- Import ruka_hand urdf file -->
     <xacro:include filename="$(find ruka)/config/ruka.urdf" />
     <!-- Import control_xacro -->
@@ -9,11 +9,5 @@
     <xacro:include filename="$(find ruka)/config/imu.ros2_control.xacro" />
     <xacro:ruka_ros2_control name="RukaSystemController" initial_positions_file="$(arg initial_positions_file)"/>
-    <!--
-    <xacro:ruka_ros2_sensor
-     name="ruka" prefix="$(arg prefix)"
-     use_mock_hardware="$(arg use_mock_hardware)"
-     mock_sensor_commands="$(arg mock_sensor_commands)" />
-    -->
-    <xacro:ruka_ros2_sensor
+     <xacro:ruka_ros2_sensor
      name="RukaSensorSee" prefix="$(arg prefix)"
       />
